File: hv-driver-push-pull-n-channel.sch (KiCad schematic (older format))
At the start: 10 parts, among them P1 CONN_01X04, P2 CONN_01X03, Q1 BSS127S-7, Q2 BSS127S-7, U1 NCP5304

Commit message: Change length to match main board and add fuse
Parts:
- added C3: C, Capacitors_SMD:C_1210, symbol C
- added F1: FUSE, Resistors_ThroughHole:Resistor_Vertical_RM5mm, symbol FUSE
- added R4: R, Resistors_SMD:R_1206, symbol R
Connections:
- wire segments 24 -> 27
Other:
- moved on the sheet: P2, R1
Changed lines of the file:
@@
 L R R1
 U 1 1 570EE021
-P 3700 1700
-F 0 "R1" V 3780 1700 50  0000 C CNN
-F 1 "10" V 3700 1700 50  0000 C CNN
-F 2 "Resistors_SMD:R_1206" V 3630 1700 50  0001 C CNN
-F 3 "" H 3700 1700 50  0000 C CNN
-	1    3700 1700
+P 3650 1700
+F 0 "R1" V 3730 1700 50  0000 C CNN
+F 1 "10" V 3650 1700 50  0000 C CNN
+F 2 "Resistors_SMD:R_1206" V 3580 1700 50  0001 C CNN
+F 3 "" H 3650 1700 50  0000 C CNN
+	1    3650 1700
 	0    1    1    0
 $EndComp
@@
 	3150 1800 3150 1900
 Wire Wire Line
-	3150 1900 3800 1900
-Wire Wire Line
 	2750 950  3400 950
-Wire Wire Line
-	3150 1600 3800 1600
-Wire Wire Line
-	3800 1600 3800 1500
 Wire Wire Line
 	1850 950  2450 950
@@
 Connection ~ 4100 1700
 Wire Wire Line
-	4800 2100 4100 2100
+	4100 2100 5400 2100
 Wire Wire Line
 	2450 2150 2050 2150
@@
 	3400 1350 3400 2150
 Connection ~ 3400 1700
-Wire Wire Line
-	3550 1700 3150 1700
 Wire Wire Line
 	3400 950  3400 1150
@@
 L CONN_01X03 P2
 U 1 1 570EF2D8
-P 5000 2000
-F 0 "P2" H 5000 2200 50  0000 C CNN
-F 1 "CONN_01X03" V 5100 2000 50  0000 C CNN
-F 2 "Pin_Headers:Pin_Header_Straight_1x03" H 5000 2000 50  0001 C CNN
-F 3 "" H 5000 2000 50  0000 C CNN
-	1    5000 2000
+P 5600 2000
+F 0 "P2" H 5600 2200 50  0000 C CNN
+F 1 "CONN_01X03" V 5700 2000 50  0000 C CNN
+F 2 "Pin_Headers:Pin_Header_Straight_1x03" H 5600 2000 50  0001 C CNN
+F 3 "" H 5600 2000 50  0000 C CNN
+	1    5600 2000
 	1    0    0    -1
 $EndComp
 Wire Wire Line
-	3850 1700 4500 1700
+	4100 1300 5000 1300
 Wire Wire Line
-	4500 1700 4500 2000
+	5000 1300 5000 1900
+Text GLabel 4900 1700 1    60   Input ~ 0
+OUT
 Wire Wire Line
-	4500 2000 4800 2000
+	3500 1700 3150 1700
 Wire Wire Line
-	4100 1300 4800 1300
+	3150 1900 3800 1900
 Wire Wire Line
-	4800 1300 4800 1900
-Text GLabel 4700 2000 1    60   Input ~ 0
-OUT
+	3150 1600 3300 1600
+Wire Wire Line
+	3300 1600 3300 1500
+Wire Wire Line
+	3300 1500 3800 1500
+$Comp
+L C C3
+U 1 1 571E5491
+P 4450 1700
+F 0 "C3" H 4475 1800 50  0000 L CNN
+F 1 "C" H 4475 1600 50  0000 L CNN
+F 2 "Capacitors_SMD:C_1210" H 4488 1550 50  0001 C CNN
+F 3 "" H 4450 1700 50  0000 C CNN
+	1    4450 1700
+	0    -1   -1   0
+$EndComp
+Wire Wire Line
+	4300 1700 3800 1700
+$Comp
+L R R4
+U 1 1 571E55F3
+P 4750 1850
+F 0 "R4" V 4830 1850 50  0000 C CNN
+F 1 "R" V 4750 1850 50  0000 C CNN
+F 2 "Resistors_SMD:R_1206" V 4680 1850 50  0001 C CNN
+F 3 "" H 4750 1850 50  0000 C CNN
+	1    4750 1850
+	1    0    0    -1
+$EndComp
+Wire Wire Line
+	4600 1700 4900 1700
+Wire Wire Line
+	4750 2000 4750 2100
+Connection ~ 4750 2100
+Wire Wire Line
+	4900 1700 4900 2000
+Connection ~ 4750 1700
+$Comp
+L FUSE F1
+U 1 1 571E9FEF
+P 5150 2000
+F 0 "F1" H 5250 2050 50  0000 C CNN
+F 1 "FUSE" H 5050 1950 50  0000 C CNN
+F 2 "Resistors_ThroughHole:Resistor_Vertical_RM5mm" H 5150 2000 50  0001 C CNN
+F 3 "" H 5150 2000 50  0000 C CNN
+	1    5150 2000
+	1    0    0    -1
+$EndComp
+Wire Wire Line
+	5000 1900 5400 1900
 $EndSCHEMATC

Commit message: Use T220 transistors and add gate resistors
Parts:
- removed Q1, Q2: BSS127S-7, TO_SOT_Packages_SMD:SOT-23, symbol Q_NMOS_GSD
- added Q1, Q2: Q_NMOS_GDS, TO_SOT_Packages_THT:TO-220_Neutral123_Vertical, symbol Q_NMOS_GDS
- added R2, R3: 10, Resistors_SMD:R_1206, symbol R
- C1: footprint Capacitors_SMD:C_1206_HandSoldering -> Capacitors_SMD:C_1206
- C2: footprint Capacitors_SMD:C_1812_HandSoldering -> Capacitors_SMD:C_1210
- D1, D2: footprint Diodes_SMD:SMA_Handsoldering -> Diodes_SMD:SMA_Standard
Changed lines of the file:
@@
 LIBS:contrib
 LIBS:valves
-LIBS:wheelerlab
 LIBS:hv-driver-push-pull-n-channel-cache
 EELAYER 25 0
@@
 Comment4 ""
 $EndDescr
-$Comp
-L Q_NMOS_GSD Q1
-U 1 1 56F2F828
-P 4000 1500
-F 0 "Q1" H 4300 1550 50  0000 R CNN
-F 1 "BSS127S-7" H 4650 1450 50  0000 R CNN
-F 2 "TO_SOT_Packages_SMD:SOT-23" H 4200 1600 50  0001 C CNN
-F 3 "" H 4000 1500 50  0000 C CNN
-	1    4000 1500
-	1    0    0    -1
-$EndComp
-$Comp
-L Q_NMOS_GSD Q2
-U 1 1 56F2F867
-P 4000 1900
-F 0 "Q2" H 4300 1950 50  0000 R CNN
-F 1 "BSS127S-7" H 4650 1850 50  0000 R CNN
-F 2 "TO_SOT_Packages_SMD:SOT-23" H 4200 2000 50  0001 C CNN
-F 3 "" H 4000 1900 50  0000 C CNN
-	1    4000 1900
-	1    0    0    -1
-$EndComp
 Text GLabel 4100 2100 0    60   Input ~ 0
 GND
@@
 F 0 "C2" V 3350 1300 50  0000 L CNN
 F 1 "0.1uF" V 3250 1250 50  0000 L CNN
-F 2 "Capacitors_SMD:C_1812_HandSoldering" H 3400 1250 50  0001 C CNN
+F 2 "Capacitors_SMD:C_1210" H 3400 1250 50  0001 C CNN
 F 3 "" H 3400 1250 50  0000 C CNN
 	1    3400 1250
@@
 F 0 "D1" H 2600 1050 50  0000 C CNN
 F 1 "D" H 2600 850 50  0000 C CNN
-F 2 "Diodes_SMD:SMA_Handsoldering" H 2600 950 50  0001 C CNN
+F 2 "Diodes_SMD:SMA_Standard" H 2600 950 50  0001 C CNN
 F 3 "" H 2600 950 50  0000 C CNN
 	1    2600 950
@@
 F 0 "C1" H 2450 1000 50  0000 L CNN
 F 1 "0.1uF" H 2300 900 50  0000 L CNN
-F 2 "Capacitors_SMD:C_1206_HandSoldering" H 2300 1050 50  0001 C CNN
+F 2 "Capacitors_SMD:C_1206" H 2300 1050 50  0001 C CNN
 F 3 "" H 2300 1050 50  0000 C CNN
 	1    2300 1050
@@
 F 0 "D2" H 2600 2250 50  0000 C CNN
 F 1 "D" H 2600 2050 50  0000 C CNN
-F 2 "Diodes_SMD:SMA_Handsoldering" H 2600 2150 50  0001 C CNN
+F 2 "Diodes_SMD:SMA_Standard" H 2600 2150 50  0001 C CNN
 F 3 "" H 2600 2150 50  0000 C CNN
 	1    2600 2150
@@
 	3500 1700 3150 1700
 Wire Wire Line
-	3150 1900 3800 1900
-Wire Wire Line
 	3150 1600 3300 1600
 Wire Wire Line
 	3300 1600 3300 1500
-Wire Wire Line
-	3300 1500 3800 1500
 $Comp
 L C C3
@@
 Wire Wire Line
 	5000 1900 5400 1900
+$Comp
+L Q_NMOS_GDS Q1
+U 1 1 57310EC3
+P 4000 1500
+F 0 "Q1" H 4300 1550 50  0000 R CNN
+F 1 "Q_NMOS_GDS" H 4650 1450 50  0000 R CNN
+F 2 "TO_SOT_Packages_THT:TO-220_Neutral123_Vertical" H 4200 1600 29  0001 C CNN
+F 3 "" H 4000 1500 60  0000 C CNN
+	1    4000 1500
+	1    0    0    -1
+$EndComp
+$Comp
+L Q_NMOS_GDS Q2
+U 1 1 57310F58
+P 4000 1900
+F 0 "Q2" H 4300 1950 50  0000 R CNN
+F 1 "Q_NMOS_GDS" H 4650 1850 50  0000 R CNN
+F 2 "TO_SOT_Packages_THT:TO-220_Neutral123_Vertical" H 4200 2000 29  0001 C CNN
+F 3 "" H 4000 1900 60  0000 C CNN
+	1    4000 1900
+	1    0    0    -1
+$EndComp
+$Comp
+L R R3
+U 1 1 5732012E
+P 3650 1900
+F 0 "R3" V 3730 1900 50  0000 C CNN
+F 1 "10" V 3650 1900 50  0000 C CNN
+F 2 "Resistors_SMD:R_1206" V 3580 1900 50  0001 C CNN
+F 3 "" H 3650 1900 50  0000 C CNN
+	1    3650 1900
+	0    1    1    0
+$EndComp
+$Comp
+L R R2
+U 1 1 57320152
+P 3650 1500
+F 0 "R2" V 3730 1500 50  0000 C CNN
+F 1 "10" V 3650 1500 50  0000 C CNN
+F 2 "Resistors_SMD:R_1206" V 3580 1500 50  0001 C CNN
+F 3 "" H 3650 1500 50  0000 C CNN
+	1    3650 1500
+	0    1    1    0
+$EndComp
+Wire Wire Line
+	3300 1500 3500 1500
+Wire Wire Line
+	3150 1900 3500 1900
 $EndSCHEMATC

Commit message: Remove gate resistors
Parts:
- removed R2, R3: 10, Resistors_SMD:R_1206, symbol R
Changed lines of the file:
@@
 	1    0    0    -1
 $EndComp
-$Comp
-L R R3
-U 1 1 5732012E
-P 3650 1900
-F 0 "R3" V 3730 1900 50  0000 C CNN
-F 1 "10" V 3650 1900 50  0000 C CNN
-F 2 "Resistors_SMD:R_1206" V 3580 1900 50  0001 C CNN
-F 3 "" H 3650 1900 50  0000 C CNN
-	1    3650 1900
-	0    1    1    0
-$EndComp
-$Comp
-L R R2
-U 1 1 57320152
-P 3650 1500
-F 0 "R2" V 3730 1500 50  0000 C CNN
-F 1 "10" V 3650 1500 50  0000 C CNN
-F 2 "Resistors_SMD:R_1206" V 3580 1500 50  0001 C CNN
-F 3 "" H 3650 1500 50  0000 C CNN
-	1    3650 1500
-	0    1    1    0
-$EndComp
 Wire Wire Line
-	3300 1500 3500 1500
+	3300 1500 3800 1500
 Wire Wire Line
-	3150 1900 3500 1900
+	3150 1900 3800 1900
 $EndSCHEMATC
